File: hw/iotAirMonitoring/interface.sch (KiCad schematic (older format))
At the start: 30 parts, among them J1 MQ-7, J13 PM1003, J2 VEML7700, J3 SHT40, J5 ML8511, J7 BMP388, J8 PMS5003, Q16 2N7002, Q17 2N7002, Q3 AO3401A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

Commit message: Create Makefile for gerbers generation, type in missing LCSC codes
Parts:
- Q16, Q17, Q4, Q6, Q8: LCSC (none) -> C8545
Changed lines of the file:
@@
 $Descr A4 11693 8268
 encoding utf-8
-Sheet 3 3
+Sheet 2 3
 Title "iotAirMonitoring"
 Date ""
@@
 F 2 "Package_TO_SOT_SMD:SOT-23" H 8950 3775 50  0001 L CIN
 F 3 "https://www.onsemi.com/pub/Collateral/NDS7002A-D.PDF" H 8750 3850 50  0001 L CNN
+F 4 "C8545" V 8750 3850 50  0001 C CNN "LCSC"
 	1    8750 3850
 	-1   0    0    -1
@@
 F 2 "Package_TO_SOT_SMD:SOT-23" H 8950 2075 50  0001 L CIN
 F 3 "https://www.onsemi.com/pub/Collateral/NDS7002A-D.PDF" H 8750 2150 50  0001 L CNN
+F 4 "C8545" V 8750 2150 50  0001 C CNN "LCSC"
 	1    8750 2150
 	-1   0    0    -1
@@
 F 2 "Package_TO_SOT_SMD:SOT-23" H 8950 5525 50  0001 L CIN
 F 3 "https://www.onsemi.com/pub/Collateral/NDS7002A-D.PDF" H 8750 5600 50  0001 L CNN
+F 4 "C8545" V 8750 5600 50  0001 C CNN "LCSC"
 	1    8750 5600
 	-1   0    0    -1
@@
 F 2 "Package_TO_SOT_SMD:SOT-23" H 5750 5725 50  0001 L CIN
 F 3 "https://www.onsemi.com/pub/Collateral/NDS7002A-D.PDF" H 5550 5800 50  0001 L CNN
+F 4 "C8545" V 5550 5800 50  0001 C CNN "LCSC"
 	1    5550 5800
 	0    1    1    0
@@
 F 2 "Package_TO_SOT_SMD:SOT-23" H 5750 6975 50  0001 L CIN
 F 3 "https://www.onsemi.com/pub/Collateral/NDS7002A-D.PDF" H 5550 7050 50  0001 L CNN
+F 4 "C8545" V 5550 7050 50  0001 C CNN "LCSC"
 	1    5550 7050
 	0    1    1    0

Commit message: Add JLCPCB assembly correction, generate gerber data
Parts:
- Q16, Q17, Q3, Q4, Q5, Q6, Q7, Q8: JLCPCB_CORRECTIONS (none) -> 0;0;180
Changed lines of the file:
@@
 F 3 "https://www.onsemi.com/pub/Collateral/NDS7002A-D.PDF" H 8750 3850 50  0001 L CNN
 F 4 "C8545" V 8750 3850 50  0001 C CNN "LCSC"
+F 5 "0;0;180" V 8750 3850 50  0001 C CNN "JLCPCB_CORRECTIONS"
 	1    8750 3850
 	-1   0    0    -1
@@
 F 3 "https://datasheet.lcsc.com/lcsc/1810171817_Alpha-&-Omega-Semicon-AO3401A_C15127.pdf" H 8650 3300 50  0001 C CNN
 F 4 "C15127" V 8650 3300 50  0001 C CNN "LCSC"
+F 5 "0;0;180" V 8650 3300 50  0001 C CNN "JLCPCB_CORRECTIONS"
 	1    8650 3300
 	0    -1   -1   0
@@
 F 3 "https://datasheet.lcsc.com/lcsc/1810171817_Alpha-&-Omega-Semicon-AO3401A_C15127.pdf" H 8650 1600 50  0001 C CNN
 F 4 "C15127" V 8650 1600 50  0001 C CNN "LCSC"
+F 5 "0;0;180" V 8650 1600 50  0001 C CNN "JLCPCB_CORRECTIONS"
 	1    8650 1600
 	0    -1   -1   0
@@
 F 3 "https://www.onsemi.com/pub/Collateral/NDS7002A-D.PDF" H 8750 2150 50  0001 L CNN
 F 4 "C8545" V 8750 2150 50  0001 C CNN "LCSC"
+F 5 "0;0;180" V 8750 2150 50  0001 C CNN "JLCPCB_CORRECTIONS"
 	1    8750 2150
 	-1   0    0    -1
@@
 F 3 "https://www.onsemi.com/pub/Collateral/NDS7002A-D.PDF" H 8750 5600 50  0001 L CNN
 F 4 "C8545" V 8750 5600 50  0001 C CNN "LCSC"
+F 5 "0;0;180" V 8750 5600 50  0001 C CNN "JLCPCB_CORRECTIONS"
 	1    8750 5600
 	-1   0    0    -1
@@
 F 3 "https://datasheet.lcsc.com/lcsc/1810171817_Alpha-&-Omega-Semicon-AO3401A_C15127.pdf" H 8650 5050 50  0001 C CNN
 F 4 "C15127" V 8650 5050 50  0001 C CNN "LCSC"
+F 5 "0;0;180" V 8650 5050 50  0001 C CNN "JLCPCB_CORRECTIONS"
 	1    8650 5050
 	0    -1   -1   0
@@
 F 3 "https://www.onsemi.com/pub/Collateral/NDS7002A-D.PDF" H 5550 5800 50  0001 L CNN
 F 4 "C8545" V 5550 5800 50  0001 C CNN "LCSC"
+F 5 "0;0;180" V 5550 5800 50  0001 C CNN "JLCPCB_CORRECTIONS"
 	1    5550 5800
 	0    1    1    0
@@
 F 3 "https://www.onsemi.com/pub/Collateral/NDS7002A-D.PDF" H 5550 7050 50  0001 L CNN
 F 4 "C8545" V 5550 7050 50  0001 C CNN "LCSC"
+F 5 "0;0;180" V 5550 7050 50  0001 C CNN "JLCPCB_CORRECTIONS"
 	1    5550 7050
 	0    1    1    0
