File: hw/iotAirMonitoring/powerManagement.sch (KiCad schematic (older format))
At the start: 40 parts, among them J10 USB_DATA, J11 PWR, J12 USB_B_Micro, J14 Battery_shield, J9 USB_C_Receptacle_USB2.0, Q10 AO3401A, Q11 2N7002, Q12 AO3401A, Q13 2N7002, Q9 AO3401A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

Commit message: Create Makefile for gerbers generation, type in missing LCSC codes
Parts:
- Q11, Q13: LCSC (none) -> C8545
- U4: LCSC (none) -> C9865
Changed lines of the file:
@@
 F 2 "Package_TO_SOT_SMD:SOT-23" H 6800 2275 50  0001 L CIN
 F 3 "https://www.fairchildsemi.com/datasheets/2N/2N7002.pdf" H 6600 2350 50  0001 L CNN
+F 4 "C8545" H 6600 2350 50  0001 C CNN "LCSC"
 	1    6600 2350
 	-1   0    0    -1
@@
 F 2 "Package_SO:SOIC-8_3.9x4.9mm_P1.27mm" H 3500 4700 50  0001 C CNN
 F 3 "https://datasheet.lcsc.com/lcsc/1808272040_Texas-Instruments-TPS54331DR_C9865.pdf" H 3500 4700 50  0001 C CNN
+F 4 "C9865" H 3500 4700 50  0001 C CNN "LCSC"
 	1    3500 4700
 	1    0    0    -1
@@
 F 2 "Package_TO_SOT_SMD:SOT-23" H 8000 4825 50  0001 L CIN
 F 3 "https://www.fairchildsemi.com/datasheets/2N/2N7002.pdf" H 7800 4900 50  0001 L CNN
+F 4 "C8545" H 7800 4900 50  0001 C CNN "LCSC"
 	1    7800 4900
 	-1   0    0    -1

Commit message: Add JLCPCB assembly correction, generate gerber data
Parts:
- added J16: Battery_voltage, Connector_PinHeader_2.54mm:PinHeader_1x01_P2.54mm_Vertical, symbol Connector_Generic:Conn_01x01
- D5, Q10, Q11, Q12, Q13, Q9, U3: JLCPCB_CORRECTIONS (none) -> 0;0;180
- U4: JLCPCB_CORRECTIONS (none) -> 0;0;270
Connections:
- net USB_VDD: no longer R1.1
- new net: J16.1 (Pin_1), R1.1
Changed lines of the file:
@@
 F 3 "https://www.fairchildsemi.com/datasheets/2N/2N7002.pdf" H 6600 2350 50  0001 L CNN
 F 4 "C8545" H 6600 2350 50  0001 C CNN "LCSC"
+F 5 "0;0;180" H 6600 2350 50  0001 C CNN "JLCPCB_CORRECTIONS"
 	1    6600 2350
 	-1   0    0    -1
@@
 F 3 "https://datasheet.lcsc.com/lcsc/1810171817_Alpha-&-Omega-Semicon-AO3401A_C15127.pdf" H 5000 1450 50  0001 C CNN
 F 4 "C15127" V 5000 1450 50  0001 C CNN "LCSC"
+F 5 "0;0;180" V 5000 1450 50  0001 C CNN "JLCPCB_CORRECTIONS"
 	1    5000 1450
 	0    -1   -1   0
@@
 F 3 "https://datasheet.lcsc.com/lcsc/1810171817_Alpha-&-Omega-Semicon-AO3401A_C15127.pdf" H 6500 1450 50  0001 C CNN
 F 4 "C15127" V 6500 1450 50  0001 C CNN "LCSC"
+F 5 "0;0;180" V 6500 1450 50  0001 C CNN "JLCPCB_CORRECTIONS"
 	1    6500 1450
 	0    1    -1   0
@@
 F 3 "https://datasheet.lcsc.com/lcsc/1808272040_Texas-Instruments-TPS54331DR_C9865.pdf" H 3500 4700 50  0001 C CNN
 F 4 "C9865" H 3500 4700 50  0001 C CNN "LCSC"
+F 5 "0;0;270" H 3500 4700 50  0001 C CNN "JLCPCB_CORRECTIONS"
 	1    3500 4700
 	1    0    0    -1
@@
 F 3 "~" H 4100 4400 50  0001 C CNN
 F 4 "C22452" V 4100 4400 50  0001 C CNN "LCSC"
+F 5 "0;0;180" V 4100 4400 50  0001 C CNN "JLCPCB_CORRECTIONS"
 	1    4100 4400
 	0    1    1    0
@@
 F 3 "http://www.advanced-monolithic.com/pdf/ds1117.pdf" H 8900 3850 50  0001 C CNN
 F 4 "C6186" H 8800 4100 50  0001 C CNN "LCSC"
+F 5 "0;0;180" H 8800 4100 50  0001 C CNN "JLCPCB_CORRECTIONS"
 	1    8800 4100
 	1    0    0    -1
@@
 F 3 "https://www.fairchildsemi.com/datasheets/2N/2N7002.pdf" H 7800 4900 50  0001 L CNN
 F 4 "C8545" H 7800 4900 50  0001 C CNN "LCSC"
+F 5 "0;0;180" H 7800 4900 50  0001 C CNN "JLCPCB_CORRECTIONS"
 	1    7800 4900
 	-1   0    0    -1
@@
 F 3 "https://datasheet.lcsc.com/lcsc/1810171817_Alpha-&-Omega-Semicon-AO3401A_C15127.pdf" H 7700 4200 50  0001 C CNN
 F 4 "C15127" V 7700 4200 50  0001 C CNN "LCSC"
+F 5 "0;0;180" V 7700 4200 50  0001 C CNN "JLCPCB_CORRECTIONS"
 	1    7700 4200
 	0    1    -1   0
@@
 Text Notes 9350 1200 0    50   ~ 0
 Optional voltage\ndivider for Vin
-Text GLabel 9200 1200 1    50   Input ~ 0
-USB_VDD
 Text GLabel 9200 2000 3    50   Input ~ 0
 GND
 Text HLabel 9300 1600 2    50   Output ~ 0
 ADC_VIN
+$Comp
+L Connector_Generic:Conn_01x01 J16
+U 1 1 61846396
+P 9200 1000
+F 0 "J16" V 9300 1050 50  0000 R CNN
+F 1 "Battery_voltage" V 9400 1250 50  0000 R CNN
+F 2 "Connector_PinHeader_2.54mm:PinHeader_1x01_P2.54mm_Vertical" H 9200 1000 50  0001 C CNN
+F 3 "~" H 9200 1000 50  0001 C CNN
+	1    9200 1000
+	0    -1   -1   0
+$EndComp
 $EndSCHEMATC
