File: hw/v1.1/mainBoard/mainBoard.kicad_sch (KiCad schematic)
At the start: 65 parts, among them J15 U.FL, J4 PROGRAMMER, J6 EN_3V3_PROGRAMMER, Q1 MMBT3904, Q14 AO3401A, Q15 2N7002, Q2 MMBT3904, SW1 PWR_ON, SW2 PWR_OFF, SW3 RESET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

Commit message: Beautify schematics in KiCad
Other:
- note added: "ESP32"
- note added: "MOUNTING HOLES"
- note added: "POWER STATUS LED"
- note added: "TEST PADS"
- note added: "USER DEFINED BUTTON"
- company: (none) -> Martin Kousal
- title: mainBoard -> iotAirMonitoring
- moved on the sheet: B2, C2, C3, H1, H2, H3, H4, JP4, JP5, R11, R12, R14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
